File: circuit design/dianlutu.sch (EAGLE design)
At the start: 36 parts, among them U1 STM32-C-64, U2 LM386N-4/NOPB, X1 MINI-USB-SCHIELD-32005-201

Commit message: update circuit
Parts:
- added C3, C4: (no value), rcl:C-USC0805
- added Q1: (no value), crystal:86SMX
- added R2: (no value), rcl:R-US_R0805
Connections:
- removed net VDDA: U1.VDDA
- new net N$10: U1.PA14/JTCK/SWCLK
- new net N$5: C3.1, Q1.2, U1.PD0-OSC_IN-CAN1RX
- new net N$6: R2.2, U1.PD1-OSC_OUT-CAN1TX
- new net N$8: U1.PA13/JTMS/SWDIO
- net 0: now also C3.2, C4.2
- net 3V: now also U1.BOOT0, U1.VDDA
- net N$7: now also C4.1, Q1.1, R2.1; no longer U1.BOOT0
